File: Hardware/pcb-stm32wl/_autosave-peripherals.kicad_sch (KiCad schematic)
At the start: 52 parts, among them J10 Qwiic, J11 Conn_02x08_Odd_Even, J13 Conn_02x08_Odd_Even, J8 DEBUG, J9 UART/I2C, Q2 PMST4401,115, SW1 USR_BTN, SW2 RESET, U10 SHTC3, U3 AD7124-8BCPZ-RL7, U6 ICM-42605, U7 MRF89XAM9AT-I/RM

Commit message: added footprints to all newly selected components.
Parts:
- R4: Distributor link (none) -> https://www.digikey.ca/en/products/detail/panasonic-electro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; Manufacturer (none) -> Panasonic Electronic Components; Manufacturer Part Number (none) -> ERJ-3EKF1002V
- R6: Distributor link (none) -> https://www.digikey.com/en/products/detail/yageo/CC0603KRX7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; Manufacturer (none) -> YAGEO; Manufacturer Part Number (none) -> CC0603KRX7R7BB104
Changed lines of the file:
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@@
 			)
 		)
-		(property "Distributor link" ""
+		(property "Distributor link" "https://www.digikey.ca/en/products/detail/panasonic-electronic-components/ERJ-3EKF1002V/196066?s=N4IgTCBcDaIKICUBSBaAzHA0gMQIwAZ8wA1EAXQF8g&&utm_adgroup=Supplier_Panasonic&utm_source=google&utm_medium=cpc&utm_campaign=EN_Supplier_Panasonic&utm_term=erj-3ekf1002v&productid=&utm_content=Supplier_Panasonic&utm_id=go_cmp-134209385_adg-128615584780_ad-648340646832_kwd-375322781237_dev-c_ext-_prd-_sig-Cj0KCQjwm7q-BhDRARIsACD6-fWoZliQAlNfDTQCSgYlGuu9Fq2tmp0oMaL9siCCUjVEH1DELbHxpMcaAo8eEALw_wcB&gad_source=1&gclid=Cj0KCQjwm7q-BhDRARIsACD6-fWoZliQAlNfDTQCSgYlGuu9Fq2tmp0oMaL9siCCUjVEH1DELbHxpMcaAo8eEALw_wcB&gclsrc=aw.ds"
 			(at 332.74 113.03 0)
 			(effects
@@
 			)
 		)
-		(property "Manufacturer" ""
+		(property "Manufacturer" "Panasonic Electronic Components"
 			(at 332.74 113.03 0)
 			(effects
@@
 			)
 		)
-		(property "Manufacturer Part Number" ""
+		(property "Manufacturer Part Number" "ERJ-3EKF1002V"
 			(at 332.74 113.03 0)
 			(effects
@@
 			)
 		)
-		(property "Distributor link" ""
-			(at 372.11 111.76 0)
-			(effects
-				(font
-					(size 1.27 1.27)
-				)
-				(hide yes)
-			)
-		)
-		(property "Manufacturer" ""
-			(at 372.11 111.76 0)
-			(effects
-				(font
-					(size 1.27 1.27)
-				)
-				(hide yes)
-			)
-		)
-		(property "Manufacturer Part Number" ""
-			(at 372.11 111.76 0)
-			(effects
+		(property "Distributor link" "https://www.digikey.com/en/products/detail/yageo/CC0603KRX7R7BB104/302822"
+			(at 372.11 111.76 0)
+			(effects
+				(font
+					(size 1.27 1.27)
+				)
+				(hide yes)
+			)
+		)
+		(property "Manufacturer" "YAGEO"
+			(at 372.11 111.76 0)
+			(effects
+				(font
+					(size 1.27 1.27)
+				)
+				(hide yes)
+			)
+		)
+		(property "Manufacturer Part Number" "CC0603KRX7R7BB104"
+			(at 372.11 111.76 0)
+			(effects
