File: Hardware/pcb-stm32wl/peripherals.kicad_sch (KiCad schematic)
At the start: 52 parts, among them J10 Qwiic, J11 Conn_02x08_Odd_Even, J13 Conn_02x08_Odd_Even, J8 DEBUG, J9 UART/I2C, Q2 PMST4401,115, SW1 USR_BTN, SW2 RESET, U10 SHTC3, U3 AD7124-8BCPZ-RL7, U6 ICM-42605, U7 MRF89XAM9AT-I/RM

Commit message: ALL BOM components have been added with manufacturing part nunmber, alongside distributor link
Parts:
- C19: Distributor link (none) -> https://www.digikey.com/en/products/detail/yageo/CC0603KRX7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; Manufacturer (none) -> YAGEO; Manufacturer Part Number (none) -> CC0603KRX7R7BB104
- R4, R6: Distributor link (none) -> https://www.digikey.ca/en/products/detail/panasonic-electro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; Manufacturer (none) -> Panasonic Electronic Components; Manufacturer Part Number (none) -> ERJ-3EKF1002V
- U6: Distributor link (none) -> https://www.digikey.ca/en/products/detail/tdk-invensense/IC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; Manufacturer (none) -> TDK InvenSense; Manufacturer Part Number (none) -> ICM-42605
- U7: Distributor link (none) -> https://www.digikey.ca/en/products/detail/microchip-technol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; Manufacturer (none) -> Microchip Technology; Manufacturer Part Number (none) -> MRF89XAM9AT-I/RM
Changed lines of the file:
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@@
 			)
 		)
-		(property "Distributor link" ""
+		(property "Distributor link" "https://www.digikey.ca/en/products/detail/tdk-invensense/ICM-42605/9953675?gclsrc=aw.ds&&utm_adgroup=General&utm_source=google&utm_medium=cpc&utm_campaign=PMax%20Shopping_Product_Zombie%20SKUs&utm_term=&productid=9953675&utm_content=General&utm_id=go_cmp-17855401585_adg-_ad-__dev-c_ext-_prd-9953675_sig-Cj0KCQjwm7q-BhDRARIsACD6-fUiamL_ZqaqPs1ju8ypbYWcq2beSpTnp8t2oy6VAJPsq3Kl4aRYmYkaAoooEALw_wcB&gad_source=1&gclid=Cj0KCQjwm7q-BhDRARIsACD6-fUiamL_ZqaqPs1ju8ypbYWcq2beSpTnp8t2oy6VAJPsq3Kl4aRYmYkaAoooEALw_wcB&gclsrc=aw.ds"
 			(at 317.5 124.46 0)
 			(effects
@@
 			)
 		)
-		(property "Manufacturer" ""
+		(property "Manufacturer" "TDK InvenSense"
 			(at 317.5 124.46 0)
 			(effects
@@
 			)
 		)
-		(property "Manufacturer Part Number" ""
+		(property "Manufacturer Part Number" "ICM-42605"
 			(at 317.5 124.46 0)
 			(effects
@@
 			)
 		)
-		(property "Distributor link" ""
+		(property "Distributor link" "https://www.digikey.com/en/products/detail/yageo/CC0603KRX7R7BB104/302822"
 			(at 398.78 95.25 0)
 			(effects
@@
 			)
 		)
-		(property "Manufacturer" ""
+		(property "Manufacturer" "YAGEO"
 			(at 398.78 95.25 0)
 			(effects
@@
 			)
 		)
-		(property "Manufacturer Part Number" ""
+		(property "Manufacturer Part Number" "CC0603KRX7R7BB104"
 			(at 398.78 95.25 0)
 			(effects
@@
 			)
 		)
-		(property "Distributor link" ""
+		(property "Distributor link" "https://www.digikey.ca/en/products/detail/panasonic-electronic-components/ERJ-3EKF1002V/196066?s=N4IgTCBcDaIKICUBSBaAzHA0gMQIwAZ8wA1EAXQF8g&&utm_adgroup=Supplier_Panasonic&utm_source=google&utm_medium=cpc&utm_campaign=EN_Supplier_Panasonic&utm_term=erj-3ekf1002v&productid=&utm_content=Supplier_Panasonic&utm_id=go_cmp-134209385_adg-128615584780_ad-648340646832_kwd-375322781237_dev-c_ext-_prd-_sig-Cj0KCQjwm7q-BhDRARIsACD6-fWoZliQAlNfDTQCSgYlGuu9Fq2tmp0oMaL9siCCUjVEH1DELbHxpMcaAo8eEALw_wcB&gad_source=1&gclid=Cj0KCQjwm7q-BhDRARIsACD6-fWoZliQAlNfDTQCSgYlGuu9Fq2tmp0oMaL9siCCUjVEH1DELbHxpMcaAo8eEALw_wcB&gclsrc=aw.ds"
 			(at 332.74 113.03 0)
 			(effects
@@
 			)
 		)
-		(property "Manufacturer" ""
+		(property "Manufacturer" "Panasonic Electronic Components"
 			(at 332.74 113.03 0)
 			(effects
@@
 			)
 		)
-		(property "Manufacturer Part Number" ""
+		(property "Manufacturer Part Number" "ERJ-3EKF1002V"
 			(at 332.74 113.03 0)
 			(effects
@@
 			)
 		)
-		(property "Distributor link" ""
+		(property "Distributor link" "https://www.digikey.ca/en/products/detail/microchip-technology/MRF89XAM9AT-I-RM/10519305"
 			(at 335.28 182.88 0)
 			(effects
@@
 			)
 		)
-		(property "Manufacturer" ""
+		(property "Manufacturer" "Microchip Technology"
 			(at 335.28 182.88 0)
 			(effects
@@
 			)
 		)
-		(property "Manufacturer Part Number" ""
+		(property "Manufacturer Part Number" "MRF89XAM9AT-I/RM"
 			(at 335.28 182.88 0)
 			(effects
@@
 			)
 		)
-		(property "Distributor link" ""
+		(property "Distributor link" "https://www.digikey.ca/en/products/detail/panasonic-electronic-components/ERJ-3EKF1002V/196066?s=N4IgTCBcDaIKICUBSBaAzHA0gMQIwAZ8wA1EAXQF8g&&utm_adgroup=Supplier_Panasonic&utm_source=google&utm_medium=cpc&utm_campaign=EN_Supplier_Panasonic&utm_term=erj-3ekf1002v&productid=&utm_content=Supplier_Panasonic&utm_id=go_cmp-134209385_adg-128615584780_ad-648340646832_kwd-375322781237_dev-c_ext-_prd-_sig-Cj0KCQjwm7q-BhDRARIsACD6-fWoZliQAlNfDTQCSgYlGuu9Fq2tmp0oMaL9siCCUjVEH1DELbHxpMcaAo8eEALw_wcB&gad_source=1&gclid=Cj0KCQjwm7q-BhDRARIsACD6-fWoZliQAlNfDTQCSgYlGuu9Fq2tmp0oMaL9siCCUjVEH1DELbHxpMcaAo8eEALw_wcB&gclsrc=aw.ds"
 			(at 372.11 111.76 0)
 			(effects
@@
 			)
 		)
-		(property "Manufacturer" ""
+		(property "Manufacturer" "Panasonic Electronic Components"
 			(at 372.11 111.76 0)
 			(effects
@@
 			)
 		)
-		(property "Manufacturer Part Number" ""
+		(property "Manufacturer Part Number" "ERJ-3EKF1002V"
 			(at 372.11 111.76 0)
 			(effects
