File: Hardware/pcb-stm32wl/_autosave-stm32wl.kicad_sch (KiCad schematic)
At the start: 20 parts, among them U5 STM32WL55CCU6, X1 32MHz, Y1 32.768KHz

Commit message: power circuitry completely wired
Parts:
- C13, C15: Distributor link (none) -> https://lcsc.com/product-detail/Multilayer-Ceramic-Capacito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; Manufacturer Part Number (none) -> CL10A475KO8NNNC
- C14, C16, C17, C18, C20, C24: Distributor link (none) -> https://lcsc.com/product-detail/Multilayer-Ceramic-Capacito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; Manufacturer Part Number (none) -> CC0402KRX7R7BB104
- C21: Distributor link (none) -> https://lcsc.com/product-detail/Others_YAGEO-CC0402FRNPO9BN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; Manufacturer Part Number (none) -> CC0402FRNPO9BN330
- C23: Distributor link (none) -> https://lcsc.com/product-detail/Multilayer-Ceramic-Capacito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; Manufacturer Part Number (none) -> CC0402JRNPO9BN470
- C34: Distributor link (none) -> https://lcsc.com/product-detail/Multilayer-Ceramic-Capacito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; Manufacturer Part Number (none) -> CC0402KRX7R7BB103
- C43: Distributor link (none) -> https://lcsc.com/product-detail/Chip-Resistor-Surface-Mount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; Manufacturer Part Number (none) -> CC0402KRX7R7BB102; URL (none) -> https://lcsc.com/product-detail/Chip-Resistor-Surface-Mount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
- C46, C49: Distributor link (none) -> https://lcsc.com/product-detail/Multilayer-Ceramic-Capacito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; Manufacturer Part Number (none) -> CC0402BRNPO9BN5R6
- FB1: Distributor link (none) -> https://lcsc.com/product-detail/Ferrite-Beads_Murata-Electr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; Manufacturer Part Number (none) -> BLM18AG601SN1D
- L10: Distributor link (none) -> https://lcsc.com/product-detail/Ferrite-Beads_Murata-Electr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; Manufacturer Part Number (none) -> BLM15HG102SN1D
- R5: Distributor link (none) -> https://lcsc.com/product-detail/Chip-Resistor-Surface-Mount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; Manufacturer Part Number (none) -> RC0402FR-07220RL
- U5: Distributor link (none) -> https://www.st.com/en/microcontrollers-microprocessors/stm3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; Manufacturer Part Number (none) -> STM32WL55CCU6
- X1: Distributor link (none) -> https://www.digikey.de/product-detail/en/TG2520SMN+32.0000M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; Manufacturer Part Number (none) -> ‎TG2520SMN 32.0000M-MCGNNM3‎
- Y1: Distributor link (none) -> https://lcsc.com/product-detail/SMD-Crystal-Resonators_Seik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; Manufacturer Part Number (none) -> X1A000061002100
Changed lines of the file:
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@@
 			)
 		)
-		(property "Distributor link" ""
+		(property "Distributor link" "https://www.st.com/en/microcontrollers-microprocessors/stm32wl55cc.html"
 			(at 86.36 86.36 0)
 			(effects
@@
 			)
 		)
-		(property "Manufacturer Part Number" ""
+		(property "Manufacturer Part Number" "STM32WL55CCU6"
 			(at 86.36 86.36 0)
 			(effects
@@
 			)
 		)
-		(property "Distributor link" ""
+		(property "Distributor link" "https://lcsc.com/product-detail/SMD-Crystal-Resonators_Seiko-Epson_X1A000061002100_Seiko-Epson-X1A000061002100_C255767.html"
 			(at 221.615 43.18 0)
 			(effects
@@
 			)
 		)
-		(property "Manufacturer Part Number" ""
+		(property "Manufacturer Part Number" "X1A000061002100"
 			(at 221.615 43.18 0)
 			(effects
@@
 			)
 		)
-		(property "Distributor link" ""
+		(property "Distributor link" "https://lcsc.com/product-detail/Multilayer-Ceramic-Capacitors-MLCC-SMD-SMT_YAGEO-CC0402BRNPO9BN5R6_C505468.html"
 			(at 215.265 51.435 0)
 			(effects
@@
 			)
 		)
-		(property "Manufacturer Part Number" ""
+		(property "Manufacturer Part Number" "CC0402BRNPO9BN5R6"
 			(at 215.265 51.435 0)
 			(effects
@@
 			)
 		)
-		(property "Distributor link" ""
+		(property "Distributor link" "https://lcsc.com/product-detail/Multilayer-Ceramic-Capacitors-MLCC-SMD-SMT_YAGEO-CC0402BRNPO9BN5R6_C505468.html"
 			(at 227.33 51.435 0)
 			(effects
@@
 			)
 		)
-		(property "Manufacturer Part Number" ""
+		(property "Manufacturer Part Number" "CC0402BRNPO9BN5R6"
 			(at 227.33 51.435 0)
 			(effects
@@
 			)
 		)
-		(property "URL" ""
+		(property "URL" "https://lcsc.com/product-detail/Chip-Resistor-Surface-Mount_YAGEO-RC0402FR-070RL_C106231.html "
 			(at 192.405 34.29 0)
 			(effects
@@
 			)
 		)
-		(property "Distributor link" ""
+		(property "Distributor link" "https://lcsc.com/product-detail/Chip-Resistor-Surface-Mount_YAGEO-RC0402FR-070RL_C106231.html "
 			(at 192.405 34.29 0)
 			(effects
@@
 			)
 		)
-		(property "Manufacturer Part Number" ""
+		(property "Manufacturer Part Number" "CC0402KRX7R7BB102"
 			(at 192.405 34.29 0)
 			(effects
@@
 			)
 		)
-		(property "Distributor link" ""
+		(property "Distributor link" "https://lcsc.com/product-detail/Multilayer-Ceramic-Capacitors-MLCC-SMD-SMT_SAMSUNG_CL10A475KO8NNNC_4-7uF-475-10-16V_C19666.html"
 			(at 32.385 56.515 0)
 			(effects
@@
 			)
 		)
-		(property "Manufacturer Part Number" ""
+		(property "Manufacturer Part Number" "CL10A475KO8NNNC"
 			(at 32.385 56.515 0)
 			(effects
@@
 			)
 		)
-		(property "Distributor link" ""
+		(property "Distributor link" "https://lcsc.com/product-detail/Multilayer-Ceramic-Capacitors-MLCC-SMD-SMT_SAMSUNG_CL10A475KO8NNNC_4-7uF-475-10-16V_C19666.html"
 			(at 18.415 32.385 0)
 			(effects
@@
 			)
 		)
-		(property "Manufacturer Part Number" ""
+		(property "Manufacturer Part Number" "CL10A475KO8NNNC"
 			(at 18.415 32.385 0)
 			(effects
@@
 			)
 		)
-		(property "Distributor link" ""
+		(property "Distributor link" "https://lcsc.com/product-detail/Multilayer-Ceramic-Capacitors-MLCC-SMD-SMT_YAGEO-CC0402KRX7R7BB104_C60474.html"
 			(at 27.94 32.385 0)
 			(effects
@@
 			)
 		)
-		(property "Manufacturer Part Number" ""
+		(property "Manufacturer Part Number" "CC0402KRX7R7BB104"
 			(at 27.94 32.385 0)
 			(effects
@@
 			)
 		)
-		(property "Distributor link" ""
+		(property "Distributor link" "https://lcsc.com/product-detail/Multilayer-Ceramic-Capacitors-MLCC-SMD-SMT_YAGEO-CC0402KRX7R7BB104_C60474.html"
 			(at 48.26 32.385 0)
 			(effects
@@
 			)
 		)
-		(property "Manufacturer Part Number" ""
+		(property "Manufacturer Part Number" "CC0402KRX7R7BB104"
 			(at 48.26 32.385 0)
 			(effects
@@
 			)
 		)
-		(property "Distributor link" ""
+		(property "Distributor link" "https://lcsc.com/product-detail/Multilayer-Ceramic-Capacitors-MLCC-SMD-SMT_YAGEO-CC0402KRX7R7BB104_C60474.html"
 			(at 37.465 32.385 0)
 			(effects
@@
 			)
 		)
-		(property "Manufacturer Part Number" ""
+		(property "Manufacturer Part Number" "CC0402KRX7R7BB104"
 			(at 37.465 32.385 0)
 			(effects
@@
 			)
 		)
-		(property "Distributor link" ""
+		(property "Distributor link" "https://lcsc.com/product-detail/Multilayer-Ceramic-Capacitors-MLCC-SMD-SMT_YAGEO-CC0402KRX7R7BB104_C60474.html"
 			(at 59.055 32.385 0)
 			(effects
@@
 			)
 		)
-		(property "Manufacturer Part Number" ""
+		(property "Manufacturer Part Number" "CC0402KRX7R7BB104"
 			(at 59.055 32.385 0)
 			(effects
@@
 			)
 		)
-		(property "Distributor link" ""
+		(property "Distributor link" "https://lcsc.com/product-detail/Chip-Resistor-Surface-Mount_YAGEO-RC0402FR-07220RL_C112291.html"
 			(at 192.405 41.91 0)
 			(effects
@@
 			)
 		)
-		(property "Manufacturer Part Number" ""
+		(property "Manufacturer Part Number" "RC0402FR-07220RL"
 			(at 192.405 41.91 0)
 			(effects
@@
 			)
 		)
-		(property "Distributor link" ""
+		(property "Distributor link" "https://lcsc.com/product-detail/Ferrite-Beads_Murata-Electronics-BLM15HG102SN1D_C76889.html"
 			(at 177.165 33.02 0)
 			(effects
@@
 			)
 		)
-		(property "Manufacturer Part Number" ""
+		(property "Manufacturer Part Number" "BLM15HG102SN1D"
 			(at 177.165 33.02 0)
 			(effects
@@
 			)
 		)
-		(property "Distributor link" ""
+		(property "Distributor link" "https://lcsc.com/product-detail/Multilayer-Ceramic-Capacitors-MLCC-SMD-SMT_YAGEO-CC0402KRX7R7BB103_C327009.html"
 			(at 167.005 40.005 0)
 			(effects
@@
 			)
 		)
-		(property "Manufacturer Part Number" ""
+		(property "Manufacturer Part Number" "CC0402KRX7R7BB103"
 			(at 167.005 40.005 0)
 			(effects
@@
 			)
 		)
-		(property "Distributor link" ""
+		(property "Distributor link" "https://lcsc.com/product-detail/Multilayer-Ceramic-Capacitors-MLCC-SMD-SMT_YAGEO-CC0402KRX7R7BB104_C60474.html"
 			(at 43.815 56.515 0)
 			(effects
@@
 			)
 		)
-		(property "Manufacturer Part Number" ""
+		(property "Manufacturer Part Number" "CC0402KRX7R7BB104"
 			(at 43.815 56.515 0)
 			(effects
@@
 			)
 		)
-		(property "Distributor link" ""
+		(property "Distributor link" "https://lcsc.com/product-detail/Ferrite-Beads_Murata-Electronics-BLM18AG601SN1D_C19330.html"
 			(at 24.13 52.07 0)
 			(effects
@@
 			)
 		)
-		(property "Manufacturer Part Number" ""
+		(property "Manufacturer Part Number" "BLM18AG601SN1D"
 			(at 24.13 52.07 0)
 			(effects
@@
 			)
 		)
-		(property "Distributor link" ""
+		(property "Distributor link" "https://www.digikey.de/product-detail/en/TG2520SMN+32.0000M-MCGNNM3/114-TG2520SMN32.0000M-MCGNNM3CT-ND/13152046?itemSeq=363783210"
 			(at 177.165 46.355 0)
 			(effects
@@
 			)
 		)
-		(property "Manufacturer Part Number" ""
+		(property "Manufacturer Part Number" "‎TG2520SMN 32.0000M-MCGNNM3‎"
 			(at 177.165 46.355 0)
 			(effects
@@
 			)
 		)
-		(property "Distributor link" ""
+		(property "Distributor link" "https://lcsc.com/product-detail/Others_YAGEO-CC0402FRNPO9BN330_C327064.html"
 			(at 67.31 55.88 0)
 			(effects
@@
 			)
 		)
-		(property "Manufacturer Part Number" ""
+		(property "Manufacturer Part Number" "CC0402FRNPO9BN330"
 			(at 67.31 55.88 0)
 			(effects
@@
 			)
 		)
-		(property "Distributor link" ""
+		(property "Distributor link" "https://lcsc.com/product-detail/Multilayer-Ceramic-Capacitors-MLCC-SMD-SMT_YAGEO-CC0402KRX7R7BB104_C60474.html"
 			(at 95.885 55.88 0)
 			(effects
@@
 			)
 		)
-		(property "Manufacturer Part Number" ""
+		(property "Manufacturer Part Number" "CC0402KRX7R7BB104"
 			(at 95.885 55.88 0)
 			(effects
@@
 			)
 		)
-		(property "Distributor link" ""
+		(property "Distributor link" "https://lcsc.com/product-detail/Multilayer-Ceramic-Capacitors-MLCC-SMD-SMT_YAGEO-CC0402JRNPO9BN470_C60137.html"
 			(at 87.63 55.88 0)
 			(effects
@@
 			)
 		)
-		(property "Manufacturer Part Number" ""
+		(property "Manufacturer Part Number" "CC0402JRNPO9BN470"
 			(at 87.63 55.88 0)
 			(effects
