File: Hardware/Revision01/Revision01_Application.kicad_sch (KiCad schematic)
At the start: 75 parts, among them J2 StrainConn, J3 StrainConn, J4 StrainConn, J5 StrainConn, J6 StrainConn, J7 StrainConn, J8 StrainConn, J9 StrainConn, Q1 PMOS, Q2 NMOS, Q3 PMOS, U3 TLV9062IDSGR, U4 LP5813BDRRR, U5 MRF89XAM9AT-I/RM, U6 ICM-45605

Commit message: Started working on PART B schematic, making small changes on PART A
ADC uncertainty calculated to be 1.22%
Added External GPIO's that may or may not use
	 start/stop, indication RGB leds

Started working on PART B schematic on ALTIUM, properly imported components with footprints
Parts:
- removed C11, C14, C3, C4, C7: 0.1uF, Capacitor_SMD:C_0805_2012Metric_Pad1.18x1.45mm_HandSolder, symbol Device:C_Small
- removed R16: 200K, Resistor_SMD:R_0603_1608Metric_Pad0.98x0.95mm_HandSolder, symbol Device:R_Small
- removed R17: 100K, Resistor_SMD:R_0603_1608Metric_Pad0.98x0.95mm_HandSolder, symbol Device:R_Small
- removed R5: 1.5K, Resistor_SMD:R_0603_1608Metric_Pad0.98x0.95mm_HandSolder, symbol Device:R_Small
- removed U3: TLV9062IDSGR, symbol Simulation_SPICE:OPAMP
- removed Uw1: INA317xxDGK, Package_SO:VSSOP-8_3x3mm_P0.65mm, symbol INA317:INA333xxDGK
- added D3: Indicication_RGB_Led, Connector_PinHeader_2.54mm:PinHeader_1x03_P2.54mm_Vertical, symbol Device:LED_RGB
- added Q4: PMOS, Package_TO_SOT_SMD:TSOT-23, symbol Simulation_SPICE:PMOS
- added R26, R27: R, symbol Device:R
- J2, J3, J4, J5, J6, J7, J8, J9: footprint 691137710003:691137710003 -> JST:JST_B3B-XH-A; Distributor link https://www.digikey.ca/en/products/detail/w-rth-elektronik/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 -> https://www.digikey.ca/en/products/detail/jst-sales-america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; Manufacturer Würth Elektronik -> JST Sales America Inc.; Manufacturer Part Number 691137710003 -> B3B-XH-A; Price per unit (none) -> 0.166
- renumbered C15 to C10, C16 to C11, C17 to C12, C18 to C13, C19 to C14, C20 to C15, C21 to C16, C22 to C17, C23 to C18, C5 to C3, C6 to C4, C8 to C5, C9 to C6, C10 to C7, C13 to C8, C12 to C9, D3 to D4, D4 to D5, D5 to D6, R11 to R10, R12 to R11, R13 to R12, R15 to R13, R18 to R15, R19 to R16, R20 to R17, R21 to R18, R22 to R19, R23 to R20, R24 to R21, R25 to R22, R26 to R23, R27 to R24, R28 to R25, R7 to R5, R8 to R6, R6 to R7, R9 to R8, R10 to R9, U4 to U3, U5 to U4, U6 to U5
Connections:
- net GND: now also R26.2, R27.2
- net U1_OUT0: now also D3.4 (BA), D3.5 (GA), D3.6 (RA)
- net U1_OUT1: now also D3.1 (RK)
- net U1_OUT2: now also D3.2 (GK)
- net U1_OUT3: now also D3.3 (BK)
- new net: Q4.2 (G), R26.1
- new net: Q4.3 (S), R27.1
- new net Vin: Q4.1 (D)
Other:
- added sheet instrumentationAmplifier.sch (instrumentationAmplifier.sch.kicad_sch)
- note added: "20mA hold 40mA trip SC branch protection"
- note added: "ADC uncertainty calculated to be 1.22% Added External GPIO's that may or may not use start/stop, indication RGB leds Started working on PART B schematic on ALTIUM, properly imported components with footprints"
- note added: "Careful of linear region"
- note added: "Low on state"
- note removed: "1.66V -> Aiming for 3.3V/2 Vref"
- note removed: "20mA hold 40mA trip"
- note removed: "INA2331/INA331/ INA2331/INA2332 Much cheaper options at cost of performance INA317 - Second best (26.4$) INA333(automotive grade 46.2$)"
- note removed: "Stimulation results: Rg = 1500K gives output range of 0.33V -> 3V"
- note removed: "input range 0.1+GNND -> VCC-0.1"
- moved on the sheet: C10, C11, C12, C3, C4, C5, C6, C7, C9, J2, J3, J4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
