File: Hardware/Revision01/_autosave-Revision01_Application.kicad_sch (KiCad schematic)
At the start: 83 parts, among them J10 StrainConn, J11 StrainConn, J12 StrainConn, J5 StrainConn, J6 StrainConn, J7 StrainConn, J8 StrainConn, J9 StrainConn, Q1 PMOS, Q2 NMOS, Q3 PMOS, U2 MRF89XAM9AT-I/RM, U3 ICM-45605

Commit message: redid ROUTING. Need to redefine layer stackup and stitching via length
Other:
- note added: "Stiching VIA Length calculation"
- moved on the sheet: C10, Q1, R17, R18, R19, R20, R21, R22, R23, R24, R25
