File: Hardware/Revision01/_autosave-Revision01.kicad_sch (KiCad schematic)
At the start: 35 parts, among them J1 Conn_01x05, J14 Conn_01x05, J2 Conn_01x02, J3 Conn_01x02, J4 Battery connector, SW1 ON/OFF_SW_SPST_LED, U1 NUCLEO-L476RG, U6 LMR51603XFDBVR

Commit message: rewired and routed ANOTHER buck converter due to LDO dropout not accounted for.
BATTERY->BUCK_7V ->5V LDO
Parts:
- L1: footprint DRA74-151-R:IND_CB_DRA74 -> 74404042151:WE-LQS_4018
Changed lines of the file:
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@@
 			)
 		)
-		(property "Footprint" "DRA74-151-R:IND_CB_DRA74"
+		(property "Footprint" "74404042151:WE-LQS_4018"
 			(at 85.09 148.59 0)
 			(effects
